File: pcb/dac.kicad_pcb (KiCad board)
At the start: 2 copper layers, 59.6 x 50.8 mm, 30 parts, among them J1 USB_to_I2S, J3 Conn_01x04_Pin, J4 AudioJack4, U1 PCM5102A, U2 LP5907MFX-3.3, U3 OPA2134PA

Commit message: update pcb
Parts:
- J3: footprint Connector_PinHeader_1.00mm:PinHeader_1x04_P1.00mm_Vertical -> Connector_PinHeader_2.54mm:PinHeader_1x04_P2.54mm_Vertical
- moved J3 2.25 mm to (98.8, 84.8)
Routing:
- net GND: track 69.6 -> 77.4 mm
- net AGND: track 99.7 -> 99.0 mm, vias 9 -> 6
